File: pcb/tritag/rev_c/tritag.sch (EAGLE design)
At the start: 47 parts, among them J1 TC2030-JLINK-NL, J2 TC2030-JLINK-NL, J3 MICRO_USB_B_HIROSE_ZX62-B-5PA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, J4 BAT_HOLE, J5 BAT_HOLE, U1 NRF51822QF, U2 TRIPOINT, U3 LTC4065, U4 MAX8887EZK33+T, X1 EPSON-FA-128

Commit message: added fundamental parts for TriTag
Parts:
- added C16, C17, C45, C46, C47, C48: 12pF, passives:CAPACITOR0201_CAP
- added C18, C21, C58: 4.7uF, passives:CAPACITOR0603_CAP
- added C19: 10uF, passives:CAPACITOR0603_CAP
- added C20, C22, C23, C24, C25, C26, C27, C28, C29, C30, C36, C37, C38, C39, C40, C57: 0.1uF, passives:CAPACITOR0201_CAP
- added C31, C32: 10pF, passives:CAPACITOR0201_CAP
- added C33, C34: 330pF, passives:CAPACITOR0201_CAP
- added C35: 0.01uF, passives:CAPACITOR0201_CAP
- added C41: 820pF, passives:CAPACITOR0201_CAP
- added C42: 27pF, passives:CAPACITOR0201_CAP
- added C43: 1.2pF, passives:CAPACITOR0201_CAP
- added C44: 18pF, passives:CAPACITOR0201_CAP
- added C49, C50, C51, C53: 100nF, passives:CAPACITOR0201_CAP
- added C52, C54: 4.7uF, passives:CAPACITOR0201_CAP
- added C55: 10nF, passives:CAPACITOR0201_CAP
- added C56: 1uF, passives:CAPACITOR0201_CAP
- added C59: 0.1uF, passives:CAPACITOR0402_CAP
- added D3: SML-LX0404SIUPGUSB, leds:SML-LX0404SIUPGUSB
- added J6: TC2030-JLINK-NL, connector:TC2030-JLINK-NL
- added R10: 16k, passives:RESISTOR0201_RES
- added R11, R12: 11k, passives:RESISTOR0201_RES
- added R13, R14, R15: 1k, passives:RESISTOR0402_RES
- added R16: 100k, passives:RESISTOR0201_RES
- added R9: 270, passives:RESISTOR0201_RES
- added SJ2, SJ3, SJ4, SJ5: SOLDERJUMPERNC2, SparkFun-Passives:SOLDERJUMPERNC2
- added T1: HHM1595A1, rf:HHM1595A1
- added TP10, TP11, TP12, TP7, TP8, TP9: TEST-POINT, headers:TEST-POINT
- added TP5, TP6: TEST_POINT_0.040IN, headers:TEST_POINT_0.040IN
- added U5: STM32F091CC, chips:STM32F091CC
- added U6: SKY13317, switches:SKY13317
- added U7: LXDC2HN18A, regulators:LXDC2HN18A
- added U8: DW1000, chips:DW1000
- added X2: 38.4M, crystals:FA-20H
- added X3: 16M, crystals:FA-20H
- C1, C10, C11, C12, C13, C14, C15, C2, C3, C4, C5, C6, C7, C8, C9: device passives:CAPACITOR -> passives:CAPACITOR0402_CAP
- J2: value TC2030-JLINK-NL -> MICRO_USB_B_HIROSE_ZX62R-B-5P(30); device connector:TC2030-JLINK-NL -> connector:MICRO_USB_B_HIROSE_ZX62R-B-5P(30)
- R3: value 560 1% -> 2k 1%
- U2: value TRIPOINT -> MCP73831; device tripoint:TRIPOINT -> chips:MCP73831
- U3: value LTC4065 -> FT232RQ; device chips:LTC4065 -> ftdichip:FT232RQ
- X1: value EPSON-FA-128 -> FA-20H; device crystals:EPSON-FA-128 -> crystals:FA-20H
Connections:
- removed net DW_INT: TP3.TP, U1.P25, U2.INTERRUPT
- removed net I2C_SCL: R5.1, TP1.TP, U1.P28, U2.SCL
- removed net I2C_SDA: R4.1, TP2.TP, U1.P29, U2.SDA
- removed net N$2: A2..ANTENNA, U2.ANT2
- removed net N$3: A3.ANTENNA, U2.ANT3
- removed net N$4: J2.SWDIO, U2.SWDIO
- removed net N$7: J2.SWDCLK, U2.SWDCLK
- removed net N$8: J2.!RESET, U2.!RESET
- new net !DW_RST: U5.PB0, U8.!RST
- new net !DW_SPI_CS: U5.PA4, U8.!SPICS
- new net !FTDI_RESET: SJ3.2, U3.!RESET
- new net !RST: SJ3.1
- new net !STM_RST: J6.!RESET, U5.!RST
- new net +1V8: C19.1, C20.1, C21.1, C24.1, U7.VOUT, U8.VDDLDOA, U8.VDDLDOD
- new net +3V3: C18.2, C31.1, C32.1, C33.1, C34.1, C35.1, C36.1, C37.1, C38.1, C39.1, C40.1, C49.1, C50.1, C51.1, C52.1, C53.1, C54.1, C55.1, C56.1, C58.1, D3.VDD, J6.VCC, U5.VBAT, U5.VDD/24, U5.VDD/48, U5.VDDA, U5.VDDIO2, U7.VIN, U8.VDDAON, U8.VDDBAT, U8.VDDIOA, U8.VDDLNA, U8.VDDPA1, U8.VDDPA2
- new net ANT_SEL1: U5.PB14, U6.V1
- new net ANT_SEL2: U5.PB13, U6.V2
- new net ANT_SEL3: U5.PB12, U6.V3
- new net D+: J2.D+, U3.USBDP
- new net D-: J2.D-, U3.USBDM
- new net DBG_RX: SJ5.2
- new net DBG_TX: SJ4.2
- new net DW_IRQ: R16.2, U5.PB2, U8.IRQ/GPIO8
- new net DW_SPI_CLK: U5.PA5, U8.SPICLK
- new net DW_SPI_MISO: U5.PA6, U8.SPIMISO
- new net DW_SPI_MOSI: U5.PA7, U8.SPIMOSI
- new net DW_SYNC: U8.SYNC/GPIO7
- new net DW_WAKEUP: U5.PB1, U8.WAKEUP
- new net EXT_I2C_SCL: R5.1, TP1.TP, U1.P28, U5.PA9
- new net EXT_I2C_SDA: R4.1, TP2.TP, U1.P29, U5.PA10
- new net FTDI_VCCIO: SJ2.2, U3.VCCIO
- new net GPIO0: TP5.TESTPOINT, U5.PB6
- new net GPIO1: TP6.TESTPOINT, U5.PB7
- new net GPIO2: TP7.TESTPOINT, U5.PB10
- new net GPIO3: TP8.TESTPOINT, U5.PB11
- new net INTERRUPT: TP3.TP, U1.P25, U5.PA2
- new net LED_BLUE: R15.2, TP10.TESTPOINT, U5.PB4
- new net LED_GREEN: R14.2, TP9.TESTPOINT, U5.PB3
- new net LED_RED: R13.2, TP11.TESTPOINT, U5.PB5
- new net N$12: T1.UNB, U6.RFC
- new net N$14: C16.2, T1.BAL/3
- new net N$16: C17.2, T1.BAL/4
- new net N$21: C41.1, R9.2
- new net N$22: C42.1, R10.2
- new net N$23: C44.1, R9.1, U8.VCOTUNE
- new net N$24: C43.1, R10.1, U8.CLKTUNE
- new net N$25: R11.2, U8.VREF
- new net N$26: R12.1, U5.PF11-BOOT0
- new net N$27: D3.G, R14.1
- new net N$28: D3.B, R15.1
- new net N$29: D3.R, R13.1
- new net OSC_IN: C47.1, U5.PF0-OSC_IN, X3.1
- new net OSC_OUT: C48.1, U5.PF1-OSC_OUT, X3.2
- new net REG_EN: U7.EN, U8.EXTON
- new net RF1: A1.ANTENNA, U6.RF1
- new net RF2: A2..ANTENNA, U6.RF2
- new net RF3: A3.ANTENNA, U6.RF3
- new net RF_N: C16.1, U8.RF_N
- new net RF_P: C17.1, U8.RF_P
- new net RXD: SJ4.1, U3.RXD
- new net STM_SWCLK: J6.SWDCLK, U5.PA14
- new net STM_SWDIO: J6.SWDIO, U5.PA13
- new net TXD: SJ5.1, U3.TXD
- new net USB_5V: J2.+5V, U3.VCC
- new net VDDCLK: C26.1, U8.VDDCLK
- new net VDDDIG: C22.1, C23.1, U8.VDDDIG, U8.VDDREG
- new net VDDIF: C29.1, U8.VDDIF
- new net VDDIO: C28.1, C57.1, U8.VDDIO/31, U8.VDDIO/42
- new net VDDMS: C25.1, U8.VDDMS
- new net VDDSYN: C27.1, U8.VDDSYN
- new net VDDVCO: C30.1, U8.VDDVCO
- new net XTAL1: C46.1, U8.XTAL1, X2.2
- new net XTAL2: C45.1, U8.XTAL2, X2.1
- net GND: now also C18.1, C19.2, C20.2, C21.2, C22.2, C23.2, C24.2, C25.2, C26.2, C27.2, C28.2, C29.2, C30.2, C31.2, C32.2, C33.2, C34.2, C35.2, C36.2, C37.2, C38.2, C39.2, C40.2, C41.2, C42.2, C43.2, C44.2, C45.2, C46.2, C47.2, C48.2, C49.2, C50.2, C51.2, C52.2, C53.2, C54.2, C55.2, C56.2, C57.2, C58.2, C59.2, J6.GND, R11.1, R12.2, R16.1, T1.GND, TP12.TESTPOINT, U2.VSS, U3.GND@1, U3.GND@2, U3.GND@A, U3.TEST, U5.GND, U5.VSS/23, U5.VSS/35, U5.VSS/47, U5.VSSA, U6.GND, U7.GND, U8.FORCEON, U8.GND, U8.TESTMODE, U8.VSSIO/32, U8.VSSIO/43, X2.GND, X3.GND; no longer U3.!EN
- net N$1: now also C59.1, U3.3V3OUT; no longer A1.ANTENNA, U2.ANT1
- net N$13: now also U2.PROG; no longer U3.PROG
- net N$5: now also U2.STAT; no longer U3.!CHRG
- net VBAT: now also U2.VBAT/3, U2.VBAT/4; no longer U3.BAT
- net VCC: now also SJ2.1; no longer J2.VCC, U2.VCC
- net VUSB: now also U2.VDD/1, U2.VDD/2; no longer U3.VCC
Other:
- note added: "BOOT0: Main Flash"
- note added: "DW1000"
- note added: "EXTERNAL SIGNALS"
- note added: "I2C: Pull-up resistor required"
- note added: "INTERRUPT: used both for waking up from STOP (USART2_TX) and STANDBY (WKUP4)"
- note added: "LED"
- note added: "Note: Additional I2C pull-up resistors required"
- note added: "PC Test Points"
- note added: "Pad Test Points"
- note added: "Pull-down for (DEEP)SLEEP"
- note added: "RF + DCDC"
- note added: "STM32F091CC"
- note added: "The following signals must be integrated into all designs using the design block:"
- note added: "TriPoint Interface"
- note added: "USB-Serial"
- note added: "VBAT: No backup"
- note added: "VDD"
- note added: "VDDA"
- note added: "VDDIO2"
- note added: "VDDLDOA"
- note added: "VDDLDOD"
- note removed: "TriPoint"

Commit message: added all relevant parts for carrier board and started schematic
Parts:
- removed J2: MICRO_USB_B_HIROSE_ZX62R-B-5P(30), connector:MICRO_USB_B_HIROSE_ZX62R-B-5P(30)
- removed LOGO1: UMICH_SOLID_SMALL, logos:UMICH_SOLID_SMALL
- added A2: ANT3216A063R2400A, chips:ANT3216A063R2400A
- added C60, C77: 4.7uF, passives:CAPACITOR0402_CAP
- added C61, C62, C63, C64, C75: 0.1uF, passives:CAPACITOR0402_CAP
- added C65, C71: 1uF, passives:CAPACITOR0402_CAP
- added C66: 100pF, passives:CAPACITOR0402_CAP
- added C67, C68, C73, C74: 12pF, passives:CAPACITOR0402_CAP
- added C69: 0.8pF, passives:CAPACITOR0402_CAP
- added C70: 0.5pF, passives:CAPACITOR0402_CAP
- added C72: 47nF, passives:CAPACITOR0402_CAP
- added C76: 10uF, passives:CAPACITOR0603_CAP
- added D5: SML-LX0404SIUPGUSB, leds:SML-LX0404SIUPGUSB
- added J7: CON_MICRO_SDDM3AT-SF-PEJM5, connector:CON_MICRO_SDDM3AT-SF-PEJM5
- added L3: 3.3nH, passives:INDUCTOR0402
- added L4: 15nH, passives:INDUCTOR0402
- added L5: 10uH, passives:INDUCTOR0603
- added R17, R18: DNP, passives:RESISTOR0201_RES
- added R19, R20: 100k, passives:RESISTOR0402_RES
- added R21, R22, R23: 10k, passives:RESISTOR0402_RES
- added R27, R28, R29: 470, passives:RESISTOR0402_RES
- added U10: NRF52840, chips:NRF52840
- added U12: SIP32510, chips:SIP32510
- added U9: LIS2DW12, chips:LIS2DW12
- added X4: 32MHz, crystals:7V-32.000MAHV-T
- added X5: 32.768kHz, crystals:ABS05-32.768KHZ-9-T
Connections:
- removed net SWDIO/!RESET: J1.SWDIO, U1.SWDIO/!RESET
- removed net USB_5V: J2.+5V, U3.VCC
- new net !NRF_CS_IMU: U10.P0.21, U9.CS
- new net !NRF_CS_SD: J7.DATA3-CD/CS_N, R22.1, U10.P0.19
- new net !RTC_IRQ1: U10.P1.13
- new net !RTC_IRQ2: U10.P1.14
- new net !RTC_IRQ3: U10.P1.15
- new net !SD_DETECT: J7.A, R20.1, U10.P0.24
- new net LED_NRF_BLUE: R29.2, U10.P0.05/AIN3
- new net LED_NRF_GREEN: R28.2, U10.P0.06
- new net LED_NRF_RED: R27.2, U10.P0.04/AIN2
- new net N$2: C63.1, U10.DEC1
- new net N$3: C71.1, C72.1, L4.1, U10.DEC4, U10.DEC6
- new net N$4: C66.1, U10.DEC3
- new net N$51: C67.2, U10.XC1, X4.2
- new net N$52: C68.2, U10.XC2, X4.1
- new net N$53: L5.2, U10.DCC
- new net N$54: L4.2, L5.1
- new net N$55: C77.1, J7.VCC, R20.2, R21.2, R22.2, R23.2, U12.VLOAD
- new net N$59: D5.R, R27.1
- new net N$60: D5.G, R28.1
- new net N$61: D5.B, R29.1
- new net N$7: C69.1, L3.2, U10.ANT
- new net N$8: A2.ANTENNA, C70.1, L3.1
- new net NRF_IMU_INT1: U10.P0.20, U9.INT1
- new net NRF_IMU_INT2: U10.P0.22, U9.INT2
- new net NRF_MISO: J7.DATA0/MISO, R23.1, U10.P1.09, U9.MISO/SA0
- new net NRF_MOSI: J7.CMD/MOSI, R21.1, U10.P0.08, U9.MOSI/SDA
- new net NRF_SCK: J7.CLK, U9.SCL/SPC
- new net NRF_SWDCLK: J1.SWDCLK, U10.SWDCLK
- new net NRF_SWDIO: J1.SWDIO, U10.SWDIO
- new net RTC_CS: U10.P1.12
- new net SCK: U10.P0.12
- new net SD_EN: R19.1, U10.P0.23, U12.EN
- new net STM_INTERRUPT: TP3.TP, U1.P25
- new net VBAT_OK: U10.P1.06
- new net VSEC: U10.P0.31/AIN7
- new net VSOL: U10.P0.30/AIN6
- new net WDI: U10.P0.02/AIN0
- new net XL1: C74.2, U10.P0.00/XL1, X5.1
- new net XL2: C73.2, U10.P0.01/XL2, X5.2
- net !RST: now also U10.P0.18
- net D+: now also J3.D+; no longer J2.D+
- net D-: now also J3.D-; no longer J2.D-
- net DBG_RX: now also U10.P0.26
- net DBG_TX: now also U10.P0.27
- net EXT_I2C_SCL: now also R17.1, U10.P0.14, U10.P1.10
- net EXT_I2C_SDA: now also R18.1, U10.P0.15, U10.P1.11
- net GND: now also A2.GND, C60.2, C61.2, C62.2, C63.2, C64.2, C65.2, C66.2, C67.1, C68.1, C69.2, C70.2, C71.2, C72.2, C73.1, C74.1, C75.2, C76.2, C77.2, J7.B, J7.GND, R19.2, U10.VBUS, U10.VSS, U10.VSS_PA, U12.GND, U9.GND, X4.GND; no longer J2.GND
- net INTERRUPT: no longer TP3.TP, U1.P25
- net SWDCLK: no longer J1.SWDCLK
- net VBAT: now also U10.P0.29/AIN5
- net VCC: now also C60.1, C61.1, C62.1, C64.1, C65.1, C75.1, C76.1, D5.VDD, R17.2, R18.2, U10.VDD, U10.VDDH, U12.VSUPP, U9.VCC, U9.VDD_IO
- net VUSB: now also U3.VCC
Other:
- note added: "Accelerometer"
- note added: "Do Not Populate I2C pull-up (NRF has internal pull-up)"
- note added: "SD Card Adapter"

Commit message: finished TriTag schematic
Parts:
- removed A1, A2., A3: TAIYO-YUDEN-AH086M, chips:TAIYO-YUDEN-AH086M
- removed B1: BAL-NRF01D3, chips:BAL-NRF01D3
- removed C61, C62, C63, C64: 0.1uF, passives:CAPACITOR0402_CAP
- removed C65, C71: 1uF, passives:CAPACITOR0402_CAP
- removed C66: 100pF, passives:CAPACITOR0402_CAP
- removed C67, C68, C73, C74: 12pF, passives:CAPACITOR0402_CAP
- removed C69: 0.8pF, passives:CAPACITOR0402_CAP
- removed C70: 0.5pF, passives:CAPACITOR0402_CAP
- removed C72: 47nF, passives:CAPACITOR0402_CAP
- removed D2: BLUE, SparkFun-LED:LED0603
- removed L3: 3.3nH, passives:INDUCTOR0402
- removed L4: 15nH, passives:INDUCTOR0402
- removed L5: 10uH, passives:INDUCTOR0603
- removed R1: 1k, passives:RESISTOR0402_RES
- removed R17, R18: DNP, passives:RESISTOR0201_RES
- removed R6: 12k, passives:RESISTOR0402_RES
- removed U10: NRF52840, chips:NRF52840
- removed X5: 32.768kHz, crystals:ABS05-32.768KHZ-9-T
- added A2.1, A5: TAIYO-YUDEN-AH086M, chips:TAIYO-YUDEN-AH086M
- added C78: 1pF, passives:CAPACITOR0402_CAP
- added C79: 1uF, passives:CAPACITOR0402_CAP
- added C80: 47nF, passives:CAPACITOR0402_CAP
- added C81, C82: 12pF, passives:CAPACITOR0402_CAP
- added L6: 10uH, passives:INDUCTOR0603
- A2: value ANT3216A063R2400A -> TAIYO-YUDEN-AH086M; device chips:ANT3216A063R2400A -> chips:TAIYO-YUDEN-AH086M
- A4: value FRACTUS-2.4GHZ-FR05-S1-N-0-102 -> ANT3216A063R2400A; device chips:FRACTUS-2.4GHZ-FR05-S1-N-0-102 -> chips:ANT3216A063R2400A
- C1: value 0.8pF -> 4.7uF; DIGIKEY (none) -> 445-5947-1-ND; MPN (none) -> C1005X5R0J475K050BC
- C12: value 1uF -> 12pF; DIGIKEY (none) -> 490-6197-1-ND; MPN (none) -> GRM1555C1H120GA01D
- C14: value 4.7uF -> 1pF; DIGIKEY (none) -> 490-6269-1-ND; MPN (none) -> GRM1555C1HR80BA01D
- C2, C3: value 12pF -> 0.1uF; DIGIKEY (none) -> 490-6328-1-ND; MPN (none) -> GRM155R71C104KA88J
- C4: value 1nF -> 0.1uF; DIGIKEY (none) -> 490-6328-1-ND; MPN (none) -> GRM155R71C104KA88J
- C5: value 2.2nF -> 0.1uF; DIGIKEY (none) -> 490-6328-1-ND; MPN (none) -> GRM155R71C104KA88J
- C6: value 47nF -> 1uF; DIGIKEY (none) -> 490-7195-1-ND; MPN (none) -> GRM155R70G105KA12D
- C60: value 4.7uF -> 820pF; DIGIKEY 445-5947-1-ND -> 445-1264-1-ND; MPN C1005X5R0J475K050BC -> C1005X7R1C473K050BC
- C7: value 0.1uF -> 100pF; DIGIKEY (none) -> 490-5922-1-ND; MPN (none) -> GRM1555C1H101JA01D
- C8: value 0.1uF -> 12pF; DIGIKEY (none) -> 490-6197-1-ND; MPN (none) -> GRM1555C1H120GA01D
- L1: value 15nH -> 3.9nH; DIGIKEY (none) -> 535-10426-1-ND; MPN (none) -> AISC-0402-3N3J-T
- L2: value 10uH -> 15nH; device passives:INDUCTOR0603 -> passives:INDUCTOR0402; DIGIKEY (none) -> 587-1521-1-ND; MPN (none) -> HK100515NJ-T
- R4, R5: value 10k -> DNP
- U1: value NRF51822QF -> NRF52840; device chips:NRF51822QF -> chips:NRF52840
- X1: value FA-20H -> 32MHz; device crystals:FA-20H -> crystals:7V-32.000MAHV-T
- X4: value 32MHz -> 32.768kHz; device crystals:7V-32.000MAHV-T -> crystals:ABS05-32.768KHZ-9-T
Connections:
- removed net !CHRG1: D2.A, R1.1
- removed net !RTC_IRQ1: U10.P1.13
- removed net !RTC_IRQ2: U10.P1.14
- removed net !RTC_IRQ3: U10.P1.15
- removed net ANTENNA: A4.ANTENNA, B1.SE, C1.1
- removed net AVDD: C12.1, C4.1, L1.1, U1.AVDD
- removed net DCC: L2.2, U1.DCC
- removed net N$3: C71.1, C72.1, L4.1, U10.DEC4, U10.DEC6
- removed net N$4: C66.1, U10.DEC3
- removed net N$51: C67.2, U10.XC1, X4.2
- removed net N$52: C68.2, U10.XC2, X4.1
- removed net N$53: L5.2, U10.DCC
- removed net N$54: L4.2, L5.1
- removed net N$7: C69.1, L3.2, U10.ANT
- removed net N$8: A2.ANTENNA, C70.1, L3.1
- removed net RTC_CS: U10.P1.12
- removed net SWDCLK: R6.2, U1.SWDCLK
- removed net WDI: U10.P0.02/AIN0
- removed net XL1: C74.2, U10.P0.00/XL1, X5.1
- removed net XL2: C73.2, U10.P0.01/XL2, X5.2
- new net XL3: C82.2, U1.P0.00/XL1, X4.1
- new net XL4: C81.2, U1.P0.01/XL2, X4.2
- net !NRF_CS_IMU: now also U1.P0.21; no longer U10.P0.21
- net !NRF_CS_SD: now also U1.P0.19; no longer U10.P0.19
- net !RST: now also U1.P0.18; no longer U10.P0.18
- net !SD_DETECT: now also U1.P0.24; no longer U10.P0.24
- net BATIN: now also U1.P1.07; no longer U1.P01/AIN2
- net DBG_RX: now also U1.P0.26; no longer U10.P0.26
- net DBG_TX: now also U1.P0.27; no longer U10.P0.27
- net EXT_I2C_SCL: now also U1.P0.14, U1.P1.10; no longer R17.1, U1.P28, U10.P0.14, U10.P1.10
- net EXT_I2C_SDA: now also U1.P0.15, U1.P1.11; no longer R18.1, U1.P29, U10.P0.15, U10.P1.11
- net GND: now also A4.GND, C12.1, C78.2, C79.2, C8.1, C80.2, C81.1, C82.1, U1.VBUS, U1.VSS, U1.VSS_PA; no longer A2.GND, B1.GND, C12.2, C61.2, C62.2, C63.2, C64.2, C65.2, C66.2, C67.1, C68.1, C69.2, C70.2, C71.2, C72.2, C73.1, C74.1, C8.2, R6.1, U1.GND, U10.VBUS, U10.VSS, U10.VSS_PA, X4.GND
- net LED_NRF_BLUE: now also U1.P0.05/AIN3; no longer U10.P0.05/AIN3
- net LED_NRF_GREEN: now also U1.P0.06; no longer U10.P0.06
- net LED_NRF_RED: now also U1.P0.04/AIN2; no longer U10.P0.04/AIN2
- net N$10: now also C7.1, U1.DEC3; no longer C2.1, U1.XC2, X1.2
- net N$15: now also C14.1, L1.2, U1.ANT; no longer C6.1, U1.DEC2
- net N$17: now also A4.ANTENNA, C78.1, L1.1; no longer C7.1, U1.DEC1
- net N$18: now also C8.2, U1.XC1, X1.2; no longer B1.ANT1, U1.ANT1
- net N$19: now also C12.2, U1.XC2, X1.1; no longer B1.ANT2, U1.ANT2
- net N$2: now also C60.1, U1.DEC5; no longer C63.1, U10.DEC1
- net N$20: now also L6.2, U1.DCC; no longer B1.VDD_PA, C5.1, U1.VDD_PA
- net N$37: now also L2.2, L6.1; no longer L1.2, L2.1
- net N$6: now also C4.1, U1.DEC1; no longer D2.C, U1.P17
- net N$9: now also C79.1, C80.1, L2.1, U1.DEC4, U1.DEC6; no longer C3.1, U1.XC1, X1.1
- net NRF_IMU_INT1: now also U1.P0.20; no longer U10.P0.20
- net NRF_IMU_INT2: now also U1.P0.22; no longer U10.P0.22
- net NRF_MISO: now also U1.P1.09; no longer U10.P1.09
- net NRF_MOSI: now also U1.P0.08; no longer U10.P0.08
- net NRF_SWDCLK: now also U1.SWDCLK; no longer U10.SWDCLK
- net NRF_SWDIO: now also U1.SWDIO; no longer U10.SWDIO
- net RF1: now also A5.ANTENNA; no longer A1.ANTENNA
- net RF2: now also A2.1.ANTENNA; no longer A2..ANTENNA
- net RF3: now also A2.ANTENNA; no longer A3.ANTENNA
- net SCK: now also U1.P0.12; no longer U10.P0.12
- net SD_EN: now also U1.P0.23; no longer U10.P0.23
- net STM_INTERRUPT: now also U1.P1.12; no longer U1.P25
- net VBAT: now also U1.P0.29/AIN5; no longer U10.P0.29/AIN5
- net VBAT_OK: now also U1.P1.06; no longer U10.P1.06
- net VCC: now also C1.1, C2.1, C3.1, C5.1, C6.1, U1.VDDH; no longer C14.1, C60.1, C61.1, C62.1, C64.1, C65.1, C8.1, R1.2, R17.2, R18.2, U10.VDD, U10.VDDH
- net VSEC: now also U1.P0.31/AIN7; no longer U10.P0.31/AIN7
- net VSOL: now also U1.P0.30/AIN6; no longer U10.P0.30/AIN6
Other:
- note added: "Antennas"
- note added: "nRF52840 BLE"
- note removed: "TriPoint Interface"
- note removed: "nRF51822 BLE"
