File: pcb/tripoint/v3p0/tripoint.sch (EAGLE design)
At the start: 70 parts, among them J2 TC2030-JLINK-NL, T1 HHM1595A1, U1 STM32F091CC, U2 DW1000, U3 SKY13317, U4 LXDC2HN18A, X1 38.4M, X2 16M

Commit message: finished silk for SquarePoint
Parts:
- renumbered TP1 to GPIO0, TP2 to GPIO1
Changed lines of the file:
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@@
 <part name="D1" library="leds" deviceset="SML-LX0404SIUPGUSB" device=""/>
 <part name="R7" library="passives" deviceset="RESISTOR" device="0402_RES" value="1k"/>
-<part name="TP1" library="headers" deviceset="TEST_POINT_0.040IN" device=""/>
-<part name="TP2" library="headers" deviceset="TEST_POINT_0.040IN" device=""/>
+<part name="GPIO0" library="headers" deviceset="TEST_POINT_0.040IN" device=""/>
+<part name="GPIO1" library="headers" deviceset="TEST_POINT_0.040IN" device=""/>
 <part name="TP3" library="headers" deviceset="TEST-POINT" device=""/>
 <part name="TP4" library="headers" deviceset="TEST-POINT" device=""/>
@@
 <instance part="D1" gate="G$1" x="124.46" y="22.86" rot="R90"/>
 <instance part="R7" gate="G$1" x="134.62" y="50.8" rot="R90"/>
-<instance part="TP1" gate="G$1" x="106.68" y="76.2" rot="R180"/>
-<instance part="TP2" gate="G$1" x="106.68" y="73.66" rot="R180"/>
+<instance part="GPIO0" gate="G$1" x="106.68" y="76.2" rot="R180"/>
+<instance part="GPIO1" gate="G$1" x="106.68" y="73.66" rot="R180"/>
 <instance part="TP3" gate="G$1" x="68.58" y="116.84" smashed="yes" rot="R270">
 <attribute name="NAME" x="67.437" y="120.396" size="1.016" layer="95" ratio="12" rot="R180" align="center-right"/>
@@
 <label x="96.52" y="76.2" size="1.27" layer="95" rot="MR180"/>
 <wire x1="96.52" y1="76.2" x2="104.14" y2="76.2" width="0.1524" layer="91"/>
-<pinref part="TP1" gate="G$1" pin="TESTPOINT"/>
+<pinref part="GPIO0" gate="G$1" pin="TESTPOINT"/>
 </segment>
 </net>
@@
 <label x="96.52" y="73.66" size="1.27" layer="95" rot="MR180"/>
 <wire x1="96.52" y1="73.66" x2="104.14" y2="73.66" width="0.1524" layer="91"/>
-<pinref part="TP2" gate="G$1" pin="TESTPOINT"/>
-</segment>
-</net>
+<pinref part="GPIO1" gate="G$1" pin="TESTPOINT"/>
+</segment>
+</net>
