File: pcb/tottag/rev_d/tottag.sch (EAGLE design)
At the start: 139 parts, among them J1 BAT_HOLE, J2 CON_MICRO_SDDM3AT-SF-PEJM5, J3 MICRO_USB_B_HIROSE_ZX62-B-5PA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, J4 TC2030-JLINK-NL, J5 TC2030-JLINK-NL, T1 HHM1595A1, U1 DW1000, U10 STM32F091CC, U2 FT232RQ, U3 LIS2DW12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

Commit message: fixed open issues for rev D; added test pads for SPI bus, added VBAT to analog pin
Parts:
- added MISO, MOSI, SPI_CLK: TPTP06SQ, testpad:TPTP06SQ
Connections:
- net DW_SPI_CLK: now also SPI_CLK.TP
- net DW_SPI_MISO: now also MISO.TP
- net DW_SPI_MOSI: now also MOSI.TP
- net VBAT: now also U7.P0.30/AIN6
Changed lines of the file:
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@@
 <part name="C68" library="passives" deviceset="CAPACITOR" device="0402_CAP" value="4.7uF"/>
 <part name="SUPPLY14" library="supply1" library_urn="urn:adsk.eagle:library:371" deviceset="GND" device=""/>
+<part name="SPI_CLK" library="testpad" library_urn="urn:adsk.eagle:library:385" deviceset="TP" device="TP06SQ" package3d_urn="urn:adsk.eagle:package:27952/1"/>
+<part name="MISO" library="testpad" library_urn="urn:adsk.eagle:library:385" deviceset="TP" device="TP06SQ" package3d_urn="urn:adsk.eagle:package:27952/1"/>
+<part name="MOSI" library="testpad" library_urn="urn:adsk.eagle:library:385" deviceset="TP" device="TP06SQ" package3d_urn="urn:adsk.eagle:package:27952/1"/>
 </parts>
 <sheets>
@@
 <wire x1="111.76" y1="68.58" x2="119.38" y2="68.58" width="0.1524" layer="91"/>
 <label x="109.22" y="68.58" size="1.27" layer="95"/>
+</segment>
+</net>
+<net name="VBAT" class="0">
+<segment>
+<pinref part="U7" gate="G$1" pin="P0.30/AIN6"/>
+<wire x1="106.68" y1="116.84" x2="111.76" y2="116.84" width="0.1524" layer="91"/>
+<label x="111.76" y="116.84" size="1.27" layer="95" xref="yes"/>
 </segment>
 </net>
@@
 <instance part="TP11" gate="G$1" x="213.36" y="172.72" rot="R180"/>
 <instance part="TP12" gate="G$1" x="213.36" y="170.18" rot="R180"/>
+<instance part="SPI_CLK" gate="G$1" x="119.38" y="129.54"/>
+<instance part="MISO" gate="G$1" x="124.46" y="127"/>
+<instance part="MOSI" gate="G$1" x="129.54" y="124.46"/>
 </instances>
 <busses>
@@
 <wire x1="60.96" y1="109.22" x2="60.96" y2="127" width="0.1524" layer="91"/>
 <wire x1="60.96" y1="127" x2="93.98" y2="127" width="0.1524" layer="91"/>
-<label x="93.98" y="127" size="1.27" layer="95" xref="yes"/>
+<label x="93.98" y="127" size="1.27" layer="95"/>
+<pinref part="SPI_CLK" gate="G$1" pin="TP"/>
+<wire x1="93.98" y1="127" x2="119.38" y2="127" width="0.1524" layer="91"/>
 </segment>
 <segment>
@@
 <wire x1="63.5" y1="109.22" x2="63.5" y2="124.46" width="0.1524" layer="91"/>
 <wire x1="63.5" y1="124.46" x2="93.98" y2="124.46" width="0.1524" layer="91"/>
-<label x="93.98" y="124.46" size="1.27" layer="95" xref="yes"/>
+<label x="93.98" y="124.46" size="1.27" layer="95"/>
+<pinref part="MISO" gate="G$1" pin="TP"/>
+<wire x1="93.98" y1="124.46" x2="124.46" y2="124.46" width="0.1524" layer="91"/>
 </segment>
 <segment>
@@
 <wire x1="66.04" y1="109.22" x2="66.04" y2="121.92" width="0.1524" layer="91"/>
 <wire x1="66.04" y1="121.92" x2="93.98" y2="121.92" width="0.1524" layer="91"/>
-<label x="93.98" y="121.92" size="1.27" layer="95" xref="yes"/>
-</segment>
-<segment>
+<label x="93.98" y="121.92" size="1.27" layer="95"/>
+<pinref part="MOSI" gate="G$1" pin="TP"/>
+<wire x1="93.98" y1="121.92" x2="129.54" y2="121.92" width="0.1524" layer="91"/>
+</segment>
+<segment>
