File: pcb/tottag/rev_d/tottag.brd (EAGLE design)
At the start: 61 x 34.5 mm, 141 parts, among them J1 BAT_HOLE, J2 CON_MICRO_SDDM3AT-SF-PEJM5, J3 MICRO_USB_B_HIROSE_ZX62-B-5PA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, J4 TC2030-JLINK-NL, J5 TC2030-JLINK-NL, T1 HHM1595A1, U1 DW1000, U10 STM32F091CC, U2 FT232RQ, U3 LIS2DW12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

Commit message: fixed open issues for rev D; added test pads for SPI bus, added VBAT to analog pin
Parts:
- added MISO, MOSI, SPI_CLK: TPTP06SQ, testpad:TP06SQ
Connections:
- net DW_SPI_CLK: now also SPI_CLK.TP
- net DW_SPI_MISO: now also MISO.TP
- net DW_SPI_MOSI: now also MOSI.TP
- net VBAT: now also U7.B9
Routing:
- net VBAT: track 18.8 -> 53.9 mm, vias 0 -> 1
- net NRF_GPIO_1: track 18.4 -> 6.43 mm
- net NRF_GPIO_0: track 20.7 -> 8.87 mm
- net +3V3: track 288.2 -> 277.5 mm
- net DW_SPI_CLK: track 13.4 -> 15.1 mm
- net DW_SPI_MOSI: track 11.9 -> 13.1 mm
- net DW_SPI_MISO: track 12.7 -> 13.4 mm

Commit message: added TotTernary logo
Parts:
- added U$1: (no value), logos:TOTTERNARY_300MIL
Changed lines of the file:
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@@
 <layers>
 <layer number="1" name="Top" color="4" fill="1" visible="yes" active="yes"/>
-<layer number="2" name="Route2" color="1" fill="3" visible="no" active="yes"/>
+<layer number="2" name="Route2" color="1" fill="3" visible="yes" active="yes"/>
 <layer number="3" name="Route3" color="4" fill="3" visible="no" active="no"/>
 <layer number="4" name="Route4" color="1" fill="4" visible="no" active="no"/>
@@
 <layer number="13" name="Route13" color="4" fill="5" visible="no" active="no"/>
 <layer number="14" name="Route14" color="1" fill="6" visible="no" active="no"/>
-<layer number="15" name="Route15" color="4" fill="6" visible="no" active="yes"/>
-<layer number="16" name="Bottom" color="1" fill="1" visible="no" active="yes"/>
+<layer number="15" name="Route15" color="4" fill="6" visible="yes" active="yes"/>
+<layer number="16" name="Bottom" color="1" fill="1" visible="yes" active="yes"/>
 <layer number="17" name="Pads" color="2" fill="1" visible="yes" active="yes"/>
 <layer number="18" name="Vias" color="2" fill="1" visible="yes" active="yes"/>
@@
 <layer number="20" name="Dimension" color="48" fill="1" visible="yes" active="yes"/>
 <layer number="21" name="tPlace" color="7" fill="1" visible="yes" active="yes"/>
-<layer number="22" name="bPlace" color="7" fill="1" visible="no" active="yes"/>
+<layer number="22" name="bPlace" color="7" fill="1" visible="yes" active="yes"/>
 <layer number="23" name="tOrigins" color="15" fill="1" visible="yes" active="yes"/>
-<layer number="24" name="bOrigins" color="15" fill="1" visible="no" active="yes"/>
+<layer number="24" name="bOrigins" color="15" fill="1" visible="yes" active="yes"/>
 <layer number="25" name="tNames" color="7" fill="1" visible="yes" active="yes"/>
-<layer number="26" name="bNames" color="7" fill="1" visible="no" active="yes"/>
+<layer number="26" name="bNames" color="7" fill="1" visible="yes" active="yes"/>
 <layer number="27" name="tValues" color="7" fill="1" visible="no" active="yes"/>
 <layer number="28" name="bValues" color="7" fill="1" visible="no" active="yes"/>
@@
 <layer number="38" name="bTest" color="7" fill="1" visible="no" active="yes"/>
 <layer number="39" name="tKeepout" color="4" fill="11" visible="yes" active="yes"/>
-<layer number="40" name="bKeepout" color="1" fill="11" visible="no" active="yes"/>
+<layer number="40" name="bKeepout" color="1" fill="11" visible="yes" active="yes"/>
 <layer number="41" name="tRestrict" color="4" fill="10" visible="yes" active="yes"/>
-<layer number="42" name="bRestrict" color="1" fill="10" visible="no" active="yes"/>
+<layer number="42" name="bRestrict" color="1" fill="10" visible="yes" active="yes"/>
 <layer number="43" name="vRestrict" color="2" fill="10" visible="no" active="yes"/>
 <layer number="44" name="Drills" color="7" fill="1" visible="no" active="yes"/>
@@
 <layer number="50" name="dxf" color="7" fill="1" visible="no" active="no"/>
 <layer number="51" name="tDocu" color="6" fill="1" visible="yes" active="yes"/>
-<layer number="52" name="bDocu" color="7" fill="1" visible="no" active="yes"/>
+<layer number="52" name="bDocu" color="7" fill="1" visible="yes" active="yes"/>
 <layer number="53" name="tGND_GNDA" color="7" fill="9" visible="no" active="no"/>
 <layer number="54" name="bGND_GNDA" color="1" fill="9" visible="no" active="no"/>
@@
 <attribute name="VALUE" x="-4.2418" y="16.7132" size="0.0254" layer="28" rot="MR0"/>
 </element>
+<element name="U$1" library="logos" package="TOTTERNARY_300MIL" value="" x="-8.89" y="6.477" rot="MR0"/>
 </elements>
 <signals>
