File: hardware/tottag/rev_e/tottag.sch (EAGLE design)
At the start: 145 parts, among them J1 MICRO_USB_B_HIROSE_ZX62-B-5PA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, J2 CON_MICRO_SDDM3AT-SF-PEJM5, J3 BAT_HOLE, J4 TC2030-JLINK-NL, J5 TC2030-JLINK-NL, T1 HHM1595A1, U1 DW1000, U10 STM32F091CC, U2 FT232RQ, U3 LIS2DW12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

Commit message: finished files for revision E - ready for shipping
Connections:
- net BATIN: now also U7.P0.30/AIN6
- net VBAT: no longer U7.P0.30/AIN6
Changed lines of the file:
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@@
-</segment>
-</net>
-<net name="VBAT" class="0">
-<segment>
-<pinref part="U7" gate="G$1" pin="P0.30/AIN6"/>
-<wire x1="106.68" y1="116.84" x2="111.76" y2="116.84" width="0.1524" layer="91"/>
-<label x="111.76" y="116.84" size="1.27" layer="95" xref="yes"/>
 </segment>
 </net>
@@
 </segment>
 </net>
+<net name="BATIN" class="0">
+<segment>
+<pinref part="U7" gate="G$1" pin="P0.30/AIN6"/>
+<wire x1="106.68" y1="116.84" x2="111.76" y2="116.84" width="0.1524" layer="91"/>
+<label x="111.76" y="116.84" size="1.27" layer="95" xref="yes"/>
+</segment>
+</net>
