File: hardware/tottag/rev_e/tottag.brd (EAGLE design)
At the start: 61 x 34.5 mm, 148 parts, among them J1 MICRO_USB_B_HIROSE_ZX62-B-5PA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, J2 CON_MICRO_SDDM3AT-SF-PEJM5, J3 BAT_HOLE, J4 TC2030-JLINK-NL, J5 TC2030-JLINK-NL, T1 HHM1595A1, U1 DW1000, U10 STM32F091CC, U2 FT232RQ, U3 LIS2DW12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

Commit message: finished review of revision E
Parts:
- moved C14 0.46 mm to (6.32, 18.4)
- moved C71 0.28 mm to (-9.70, 19.8)
- moved C46 0.28 mm to (-8.46, 19.5)
Routing:
- net GND: track 160.7 -> 159.1 mm, vias 365 -> 366

Commit message: finished files for revision E - ready for shipping
Parts:
- moved C59 0.48 mm to (-16.7, 18.2)
Connections:
- net BATIN: now also U7.B9
- net VBAT: no longer U7.B9
Routing:
- net BATIN: track 4.55 -> 52.3 mm, vias 0 -> 2
- net VBAT: track 53.9 -> 18.8 mm, vias 1 -> 0
- net GND: track 159.1 -> 158.1 mm, vias 366 -> 367

Commit message: updated revision E - ready for shipping
Parts:
- moved A4 4.16 mm to (24.7, 17.8)
- moved X3 2.59 mm to (13.0, 24.5)
- moved C8 2.57 mm to (13.0, 26.6)
- moved C2 2.52 mm to (20.2, 20.2), turned to 90 degrees
- moved C9 2.52 mm to (10.4, 24.5)
- moved C55 1.96 mm to (13.6, 22.8), turned to 0 degrees
- moved C30 1.85 mm to (13.6, 21.9), turned to 0 degrees
- moved TP14 1.75 mm to (8.00, 25.2)
- moved C18 1.47 mm to (16.8, 20.9)
- moved L1 1.43 mm to (18.7, 19.7), turned to 180 degrees
- moved TP13 1.37 mm to (6.22, 25.2)
- moved C1 0.55 mm to (17.3, 20.2), turned to 90 degrees
Routing:
- net GND: track 158.1 -> 165.3 mm, vias 367 -> 386
- net N$17: track 2.86 -> 4.84 mm
- net NRF_SWDIO: track 15.7 -> 17.5 mm
- net N$19: track 8.12 -> 6.50 mm
- net N$18: track 7.53 -> 6.09 mm
- net NRF_SWDCLK: track 16.8 -> 15.6 mm
- net NRF_GPIO_0: track 8.87 -> 8.06 mm
- net NRF_GPIO_1: track 6.43 -> 5.63 mm
- net +3V3: track 218.1 -> 217.9 mm, vias 25 -> 24
- added copper zone on layer 16, net N$36
- added copper zone on layer 1, net N$38
- added copper zone on layer 15, net N$39
- added copper zone on layer 2, net N$40
- removed copper zone on layer 15, net N$31
- removed copper zone on layer 16, net N$31
- removed copper zone on layer 2, net N$31
Other:
- outline, holes or cut-outs redrawn
