File: hardware/tottag/rev_h/tottag.brd (EAGLE design)
At the start: 68.1 x 39.6 mm, 216 parts, among them J1 USB4110-GF-A, J2 DM3AT-SF-PEJM5, J3 TC2030-JLINK-NL-2SIDE, J4 TC2030-JLINK-NL-2SIDE, J5 MOLEX-PICO-SPOX-3SIDE, Q1 CSD75207W15, Q2 CSD75207W15, T1 HHM1595A1, U1 DW1000, U10 STM32F091CC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

Commit message: rev_h: renumber passives
Parts:
- C66, C67: value 470nF -> 0.1uF
- C68: value 1uF -> 0.1uF
- C69, C70: value 1uF -> 470nF
- C76, C77, C78, C79: value 4.7uF -> 1uF
- C87: value 1uF -> 4.7uF
- C88, C89, C90: value 10uF -> 4.7uF; device passives:0603_CAP -> passives:0402_CAP
- C92: value 47uF -> 10uF
- C93, C94: value 0.1uF -> 10uF; device passives:0402_CAP -> passives:0603_CAP
- C95: value 0.1uF -> 47uF; device passives:0402_CAP -> passives:0603_CAP
- R25, R26: value 11k -> 10k
- R27: value 16k -> 11k
- R28: value 100k -> 11k
- R29: value 100k -> 16k
- R35: value 3.3M -> 100k
- R36: value 10M -> 100k
- R37: value DNP -> 3.3M
- R38: value 10k -> 10M
- R39: value 10k -> DNP
- moved R39 46.4 mm to (-25.8, 17.1), turned to 270 degrees
- moved C76 45.9 mm to (33.3, 27.1), turned to 90 degrees
- moved R7 45.1 mm to (-15.5, -3.56), turned to 270 degrees
- moved R10 43.1 mm to (21.4, 18.7), turned to 90 degrees
- moved C74 39.5 mm to (21.2, 23.4), turned to 180 degrees
- moved R25 34.5 mm to (19.1, 11.8)
- moved C73 32.5 mm to (2.57, 16.5)
- moved C82 31.8 mm to (-13.0, 27.7), turned to 180 degrees
- moved C91 31.6 mm to (-18.2, 10.9), turned to 270 degrees
- moved C95 31.6 mm to (-9.53, 21.2)
- moved R34 31.4 mm to (-13.0, 29.9), turned to 0 degrees
- moved C92 31.2 mm to (6.38, -5.64)
- moved C75 30.1 mm to (3.45, 2.13)
- moved R38 29.8 mm to (-7.32, 25.6), turned to 180 degrees
- moved C87 27.8 mm to (-3.38, 7.70), turned to 90 degrees
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Connections:
- net !NRF_CS_RTC: now also R36.2; no longer R34.2
- net !NRF_CS_SD: now also R33.1; no longer R31.1
- net !SD_DETECT: now also R31.1; no longer R29.1
- net +1V8: now also C84.1, C91.1; no longer C80.1, C88.1
- net +3V3: now also C66.1, C74.1, C76.1, C85.1, C86.1, C88.1, R25.1, R26.1, R36.1, R7.1; no longer C70.1, C77.1, C82.1, C84.1, C92.1, C93.1, R10.1, R34.1, R38.1, R39.1
- net BATIN: now also R37.1, R38.2; no longer R35.1, R36.2
- net BQ_AC1: now also C69.2; no longer C66.2
- net BQ_AC2: now also C70.2; no longer C67.2
- net BQ_CLAMP1: now also C69.1; no longer C66.1
- net BQ_CLAMP2: now also C70.1; no longer C67.1
- net BQ_RECT: now also C92.1, C93.1; no longer C89.1, C90.1
- net DW_IRQ: now also R35.2; no longer R33.2
- net GND: now also C66.2, C67.2, C72.2, C75.1, R27.1, R30.2, R35.1, R38.1, R39.1; no longer C69.2, C70.2, C72.1, C75.2, R25.1, R26.2, R33.1, R36.1, R37.1
- net LED_NRF_BLUE: now also R10.2; no longer R9.2
- net LED_NRF_BLUE_COMM: now also R10.1; no longer R9.1
- net LED_NRF_GREEN: now also R9.2; no longer R8.2
- net LED_NRF_GREEN_COMM: now also R9.1; no longer R8.1
- net LED_NRF_RED: now also R8.2; no longer R7.2
- net LED_NRF_RED_COMM: now also R8.1; no longer R7.1
- net LSM_SENSEHUB_SCL: now also R26.2; no longer R39.2
- net LSM_SENSEHUB_SDA: now also R25.2; no longer R38.2
- net N$12: now also R29.2; no longer R27.2
- net N$16: now also R29.1; no longer R27.1
- net N$21: now also R27.2; no longer R25.2
- net N$22: now also R28.1; no longer R26.1
- net N$33: now also C67.1; no longer C94.1
- net N$49: now also R39.2; no longer R37.2
- net N$54: now also R7.2; no longer R10.2
- net NRF_DECAP46: now also C72.1; no longer C69.1
- net NRF_DECUSB: now also C89.1; no longer C85.1
- net NRF_SPI2_MISO: now also R34.1; no longer R32.1
- net NRF_SPI2_MOSI: now also R32.1; no longer R30.1
- net SD_EN: now also R30.1; no longer R28.1
- net VBAT: now also C78.1, R37.2; no longer C75.1, R35.2
- net VBAT_SWITCHED: now also C80.1; no longer C76.1
- net VCC_SDCARD: now also C82.1, R33.2, R34.2; no longer C78.1, R29.2, R30.2
- net VQI: now also C77.1, C94.1; no longer C74.1, C91.1
- net VUSB: now also C75.2; no longer C72.2
- net VUSB_NRF: now also C90.1; no longer C86.1
