File: hardware/Apollo4-BluePlus-Module/rev_b/Apollo4-BluePlus-Module_rev_b_v7.sch (EAGLE design)
At the start: 102 parts, among them J1 TC2030-JLINK-NL-2SIDE, J2 TC2030-JLINK-NL-2SIDE, P1 CASTELLATION4L, P10 CASTELLATION4L, P11 CASTELLATION4L, P12 CASTELLATION4L, P13 CASTELLATION4L, P14 CASTELLATION4L, P15 CASTELLATION4L, P18 CASTELLATION4L, P19 CASTELLATION4L, P2 CASTELLATION4L, P20 CASTELLATION4L, P21 CASTELLATION4L, P22 CASTELLATION4L, P23 CASTELLATION4L, P24 CASTELLATION4L, P25 CASTELLATION4L, P26 CASTELLATION4L, P27 CASTELLATION4L, P28 CASTELLATION4L, P29 CASTELLATION4L, P3 CASTELLATION4L, P30 CASTELLATION4L, P31 CASTELLATION4L, P32 CASTELLATION4L, P33 CASTELLATION4L, P34 CASTELLATION4L, P35 CASTELLATION4L, P36 CASTELLATION4L, P37 CASTELLATION4L, P38 CASTELLATION4L, P39 CASTELLATION4L, P4 CASTELLATION4L, P40 CASTELLATION4L, P41 CASTELLATION4L, P42 CASTELLATION4L, P43 CASTELLATION4L, P44 CASTELLATION4L, P45 CASTELLATION4L, P46 CASTELLATION4L, P47 CASTELLATION4L, P48 CASTELLATION4L, P5 CASTELLATION4L, P6 CASTELLATION4L, P7 CASTELLATION4L, P8 CASTELLATION4L, P9 CASTELLATION4L, U1 APOLLO4_BLUE_PLUS_SOC_KBR, X1 TXC-9HT12, X2 ABM12W

Commit message: ap4bp-mod-rev_b: remove RF test switch
Parts:
- removed S4: MM8030-2610, switches:MM8030-2610
Connections:
- removed net N$18: L4.2, S4G$1.IN
- net AGND: no longer S4G$2.GND
- net BLE_RFOUT: now also L4.2; no longer S4G$1.A
Changed lines of the file:
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@@
 <part name="TP2" library="headers" deviceset="TEST-POINT" device="" value="VDDP"/>
 <part name="TP3" library="headers" deviceset="TEST-POINT" device="" value="VDDF"/>
-<part name="S4" library="switches" library_urn="urn:adsk.eagle:library:20878764" deviceset="MM8030-2610" device="" package3d_urn="urn:adsk.eagle:package:40585162/2"/>
 <part name="L3" library="Inductor" deviceset="L" device="CHIP-0402(1006-METRIC)" package3d_urn="urn:adsk.eagle:package:16378468/1" technology="_" value="2.0nH">
 <spice>
@@
 </part>
 <part name="SJ1" library="jumper" library_urn="urn:adsk.eagle:library:252" deviceset="SJ" device="" package3d_urn="urn:adsk.eagle:package:15471/1"/>
-<part name="AGND1" library="supply1" library_urn="urn:adsk.eagle:library:371" deviceset="AGND" device=""/>
 <part name="AGND2" library="supply1" library_urn="urn:adsk.eagle:library:371" deviceset="AGND" device=""/>
 <part name="CX5" library="Capacitor" deviceset="C" device="CHIP-0402(1005-METRIC)" package3d_urn="urn:adsk.eagle:package:16290895/2" technology="_" value="DNP">
@@
 <attribute name="NAME" x="135.255" y="7.62" size="1.016" layer="95" ratio="12" rot="R180" align="center-right"/>
 </instance>
-<instance part="S4" gate="G$1" x="238.76" y="40.64" smashed="yes">
-<attribute name="NAME" x="233.68" y="38.1" size="1.27" layer="95"/>
-<attribute name="VALUE" x="233.68" y="35.56" size="1.27" layer="96"/>
-</instance>
-<instance part="S4" gate="G$2" x="243.84" y="38.1" smashed="yes"/>
 <instance part="L3" gate="G$1" x="205.74" y="40.64" smashed="yes">
 <attribute name="NAME" x="205.74" y="43.18" size="1.778" layer="95" align="center"/>
@@
 <attribute name="NAME" x="53.086" y="160.02" size="1.778" layer="95" rot="R90"/>
 <attribute name="VALUE" x="53.086" y="157.734" size="1.778" layer="96" rot="R270" align="top-left"/>
-</instance>
-<instance part="AGND1" gate="VR1" x="238.76" y="33.02" smashed="yes">
-<attribute name="VALUE" x="238.76" y="32.004" size="1.778" layer="96" align="top-center"/>
 </instance>
 <instance part="AGND2" gate="VR1" x="187.96" y="25.4" smashed="yes">
@@
 </segment>
 </net>
-<net name="N$18" class="2">
-<segment>
+<net name="BLE_RFOUT" class="2">
+<segment>
+<wire x1="231.14" y1="40.64" x2="233.68" y2="40.64" width="0.1524" layer="91"/>
+<label x="233.68" y="40.64" size="1.27" layer="95" font="fixed" xref="yes"/>
 <pinref part="L4" gate="G$1" pin="2"/>
-<wire x1="231.14" y1="40.64" x2="233.68" y2="40.64" width="0.1524" layer="91"/>
-<pinref part="S4" gate="G$1" pin="IN"/>
-</segment>
-</net>
-<net name="BLE_RFOUT" class="2">
-<segment>
-<pinref part="S4" gate="G$1" pin="A"/>
-<wire x1="243.84" y1="43.18" x2="246.38" y2="43.18" width="0.1524" layer="91"/>
-<wire x1="246.38" y1="43.18" x2="246.38" y2="45.72" width="0.1524" layer="91"/>
-<label x="246.38" y="45.72" size="1.27" layer="95" font="fixed" rot="R90" xref="yes"/>
 </segment>
 </net>
@@
 <net name="AGND" class="0">
 <segment>
-<pinref part="S4" gate="G$2" pin="GND"/>
-<wire x1="241.3" y1="38.1" x2="238.76" y2="38.1" width="0.1524" layer="91"/>
-<wire x1="238.76" y1="38.1" x2="238.76" y2="35.56" width="0.1524" layer="91"/>
-<pinref part="AGND1" gate="VR1" pin="AGND"/>
-</segment>
-<segment>
 <pinref part="C12" gate="G$1" pin="2"/>
