File: hardware/tottag/rev_n/rev_n v28.sch (EAGLE design)
At the start: 197 parts, among them J2 TC2030-JLINK-NL-2SIDE, J3 TC2030-JLINK-NL-2SIDE, J4 MOLEX-PICO-SPOX-3SIDE, Q1 CSD75207W15, Q2 MOSFET-NCHANNELXFDN-3, U1 APOLLO4_BLUE_PLUS_SOC_KBR, U2 DW3110, U3 BQ24040, U4 BQ51013B, U5 W25N01GWZEIG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

Commit message: bump candidate hw rev
Parts:
- removed J3: TC2030-JLINK-NL-2SIDE, connector:TC2030-JLINK-NL-2SIDE
- removed R21: 10k, passives:RESISTOR0402_RES
- removed U5: W25N01GWZEIG, Quorvo:W25N01GWZEIG
- added J1: TC2030-JLINK-NL-2SIDE, connector:TC2030-JLINK-NL-2SIDE
- added RX2: DNP, passives:RESISTOR0603_RES
- added U8: AS5FXXX04SND, Quorvo:AS5FXXX04SND
Connections:
- net N$1 renamed USB_CC2
- net N$13 renamed USB_CC1
- removed net N$4: C31.1, U6.VDDIO
- net +1V8: now also C31.1, J1.VTREF, RX2.2, U6.VDDIO, U8.VCC; no longer J2.VTREF, R21.2, U5.VCC
- net AP4_!RESET: now also J1.!RESET; no longer J2.!RESET
- net AP4_GP06/TT_FLASH_!HOLD_IO3: now also U8.!HOLD!/SIO3; no longer U5.!HOLD
- net AP4_GP30/TT_FLASH_!WP: now also U8.!WP!/SIO2; no longer U5.!WP
- net AP4_GP47/TT_FLASH_SCK: now also U8.SCLK; no longer U5.CLK
- net AP4_GP48/TT_FLASH_PDI_IO0: now also U8.SI/SIO0; no longer U5.DI
- net AP4_GP49/TT_FLASH_PDO_IO1: now also U8.SO/SIO1; no longer U5.DO
- net AP4_GP69/TT_FLASH_!CS: now also RX2.1, U8.!CS; no longer R21.1, U5.!CS
- net AP4_GP80/SWTRACE0: now also J2.SWDIO; no longer J3.SWDIO
- net AP4_GP81/SWTRACE1: now also J2.SWDCLK; no longer J3.SWDCLK
- net AP4_GP82/SWTRACE2: now also J2.SWO; no longer J3.SWO
- net AP4_GP83/SWTRACE3: now also J2.!RESET; no longer J3.!RESET
- net AP4_SWDCLK: now also J1.SWDCLK; no longer J2.SWDCLK
- net AP4_SWDIO: now also J1.SWDIO; no longer J2.SWDIO
- net AP4_SWO: now also J1.SWO; no longer J2.SWO
- net AP4_SWTRACECLK: now also J2.VTREF; no longer J3.VTREF
- net GND: now also J1.GND, U8.GND; no longer J3.GND, U5.GND
Other:
- note added: "Sup 1.7 - 1.98 V Qui 30 µA Max 30 mA"
- note removed: "Sup 1.7 - 1.95 V Qui 10 µA Max 35 mA +CS PU 0.2mA"
- moved on the sheet: C35, J2
