File: hardware/tottag/rev_n/rev_n_v64.brd (EAGLE design)
At the start: 68.1 x 36.9 mm, 197 parts, among them J2 TC2030-JLINK-NL-2SIDE, J3 TC2030-JLINK-NL-2SIDE, J4 MOLEX-PICO-SPOX-3SIDE, Q1 CSD75207W15, Q2 MOSFET-NCHANNELXFDN-3, U1 APOLLO4_BLUE_PLUS_SOC_KBR, U2 DW3110, U3 BQ24040, U4 BQ51013B, U5 W25N01GWZEIG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

Commit message: bump candidate hw rev
Parts:
- removed J3: TC2030-JLINK-NL-2SIDE, connector:TC2030-IDC-NL-2SIDE
- removed R21: 10k, passives:0402_RES
- removed U5: W25N01GWZEIG, Quorvo:WSON127P800X600X80-9T430X340N
- added J1: TC2030-JLINK-NL-2SIDE, connector:TC2030-IDC-NL-2SIDE
- added RX2: DNP, passives:0603-RES
- added U8: AS5FXXX04SND, Quorvo:AS5FXXXXXXXX-XXLXN
- moved C35 21.9 mm to (12.6, 11.1), turned to 0 degrees
- moved J2 19.2 mm to (6.48, 26.5), turned to 90 degrees
- moved RX5 11.7 mm to (31.2, 5.08), turned to 270 degrees
- moved RX9 6.26 mm to (27.9, 7.62), flipped to the bottom, turned to 45 degrees
- moved RZ12 3.11 mm to (23.4, 8.23), turned to 180 degrees
- moved RX8 1.10 mm to (21.3, 7.15)
- moved R34 1.02 mm to (-22.0, 29.0)
- moved R16 0.91 mm to (24.0, 6.50)
- moved C36 0.62 mm to (25.5, 6.91)
- moved D3 0.61 mm to (12.3, 13.6)
- moved RZ9 0.59 mm to (13.2, 24.7)
- moved RZ7 0.55 mm to (12.0, 24.7)
- moved RZ6 0.52 mm to (10.7, 24.7)
- moved RZ11 0.51 mm to (10.6, 14.8)
- moved C76 0.51 mm to (13.7, 13.6)
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Connections:
- net N$1 renamed USB_CC2
- net N$13 renamed USB_CC1
- removed net N$4: C31.1, U6.28
- net +1V8: now also C31.1, J1.1, J1.B1, RX2.2, U6.28, U8.8; no longer J2.1, J2.B1, R21.2, U5.8
- net AP4_!RESET: now also J1.3, J1.B3; no longer J2.3, J2.B3
- net AP4_GP06/TT_FLASH_!HOLD_IO3: now also U8.7; no longer U5.7
- net AP4_GP30/TT_FLASH_!WP: now also U8.3; no longer U5.3
- net AP4_GP47/TT_FLASH_SCK: now also U8.6; no longer U5.6
- net AP4_GP48/TT_FLASH_PDI_IO0: now also U8.5; no longer U5.5
- net AP4_GP49/TT_FLASH_PDO_IO1: now also U8.2; no longer U5.2
- net AP4_GP69/TT_FLASH_!CS: now also RX2.1, U8.1; no longer R21.1, U5.1
- net AP4_GP80/SWTRACE0: now also J2.2, J2.B2; no longer J3.2, J3.B2
- net AP4_GP81/SWTRACE1: now also J2.4, J2.B4; no longer J3.4, J3.B4
- net AP4_GP82/SWTRACE2: now also J2.6, J2.B6; no longer J3.6, J3.B6
- net AP4_GP83/SWTRACE3: now also J2.3, J2.B3; no longer J3.3, J3.B3
- net AP4_SWDCLK: now also J1.4, J1.B4; no longer J2.4, J2.B4
- net AP4_SWDIO: now also J1.2, J1.B2; no longer J2.2, J2.B2
- net AP4_SWO: now also J1.6, J1.B6; no longer J2.6, J2.B6
- net AP4_SWTRACECLK: now also J2.1, J2.B1; no longer J3.1, J3.B1
- net GND: now also J1.5, J1.B5, U8.4; no longer J3.5, J3.B5, U5.4
Routing:
- net +1V8: track 102.5 -> 215.5 mm, vias 33 -> 34
- net GND: track 152.5 -> 223.7 mm, vias 331 -> 322
- net VBAT: track 14.6 -> 38.5 mm
- net AP4_GP06/TT_FLASH_!HOLD_IO3: track 49.4 -> 25.6 mm, vias 6 -> 5
- net AP4_GP30/TT_FLASH_!WP: track 23.3 -> 40.9 mm, vias 2 -> 5
- net AP4_GP49/TT_FLASH_PDO_IO1: track 18.1 -> 31.5 mm, vias 1 -> 4
- net AP4_!RESET: track 15.7 -> 23.5 mm
- net AP4_GP47/TT_FLASH_SCK: track 22.8 -> 27.3 mm, vias 1 -> 3
- net AP4_GP48/TT_FLASH_PDI_IO0: track 24.9 -> 20.8 mm, vias 4 -> 5
- net AP4_GP08/TT_9DOF_H_SCL/SCK/RX: track 30.4 -> 26.3 mm, vias 3 -> 2
- net AP4_GP25/TT_RFSW_V2: track 36.8 -> 40.8 mm
- net N$4: track 3.86 -> 0.00 mm, vias 1 -> 0
- net AP4_SWDIO: track 23.2 -> 20.4 mm
- net BNO_PS1: track 8.92 -> 6.60 mm, vias 0 -> 1
- net AP4_GP09/TT_9DOF_H_SDA/H_MISO/TX: track 27.7 -> 25.7 mm
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Other:
- board text added: "2024-09"
- board text added: "Parts U1 and U2 are BGAs with 4mm micro vias in pads. Okay to plug any/all vias in design."
- board text added: "XXX IGNORE FOR REV-K+ ; UNUSED XXX One 90Ω differential pair USB PHY - Routed as edge-coupled external - Conductor Width = 6 mil - Conductor Spacing = 12 mil - Conductor Height = 4.725 mil [0.12mm] - Er=4.5 - Modeled Zdiff ~= 90.05 Ω XXX IGNORE FOR REV-K ; UNUSED XXX"
- board text removed: "2024-08"
- board text removed: "Parts U1 and U2 are BGAs with 4mm micro vias in pads. Okay to plugs any/all vias in design."
- board text removed: "XXX IGNORE FOR REV-K+ ; UNUSED XXX One 90Ω differential pair USB PHY - Routed as edge-coupled external - Conductor Width = 6 mil - Conductor Spacing = 12 mil - Conductor Height = 4.725 mil [0.12mm] - Er=4.5 - Modeled Zdiff ~= 90.05 Ω Traces U1-P20,P21(Castellations) XXX IGNORE FOR REV-K ; UNUSED XXX"
