File: hardware/tottag/rev_n/rev_n v31.sch (EAGLE design)
At the start: 197 parts, among them J1 TC2030-JLINK-NL-2SIDE, J2 TC2030-JLINK-NL-2SIDE, J4 MOLEX-PICO-SPOX-3SIDE, Q1 CSD75207W15, Q2 MOSFET-NCHANNELXFDN-3, U1 APOLLO4_BLUE_PLUS_SOC_KBR, U2 DW3110, U3 BQ24040, U4 BQ51013B, U6 BNO086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

Commit message: update hw draft
Parts:
- C1: MPN C0402C159C5GAC7867 -> C0402C159C5GACTU
- L7: MANUFACTURER Central Technologies -> Murata; MPN CTTF0402F-2N0B -> LQG15HS2N0B02D
- L8: MANUFACTURER Central Technologies -> Murata; MPN CTTF0402F-2N2B -> LQG15HN2N2B02D
- X4: FREQ (none) -> 38.4 MHz; MANUFACTURER (none) -> TXC; MPN (none) -> 8Y38472012
Changed lines of the file:
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@@
 </spice>
 <attribute name="DESCRIPTION" value="FIXED IND 2.0NH0.1NH SMD"/>
-<attribute name="MANUFACTURER" value="Central Technologies"/>
-<attribute name="MPN" value="CTTF0402F-2N0B"/>
+<attribute name="MANUFACTURER" value="Murata"/>
+<attribute name="MPN" value="LQG15HS2N0B02D"/>
 <attribute name="TOLERANCE" value="+/- 0.1 nH"/>
 </part>
@@
 </spice>
 <attribute name="DESCRIPTION" value="FIXED IND 2.2NH0.1NH SMD"/>
-<attribute name="MANUFACTURER" value="Central Technologies"/>
-<attribute name="MPN" value="CTTF0402F-2N2B"/>
+<attribute name="MANUFACTURER" value="Murata"/>
+<attribute name="MPN" value="LQG15HN2N2B02D"/>
 <attribute name="TOLERANCE" value="+/- 0.1 nH"/>
 </part>
@@
 <attribute name="DESCRIPTION" value="CAP CER 1.5PF 50V C0G/NP0 0402"/>
 <attribute name="MANUFACTURER" value="KEMET"/>
-<attribute name="MPN" value="C0402C159C5GAC7867"/>
+<attribute name="MPN" value="C0402C159C5GACTU"/>
 <attribute name="TEMPCOEFF" value="NP0"/>
 <attribute name="TOLERANCE" value="+/- 0.25pF"/>
@@
 <attribute name="MPN" value="CL05A104KP5NNNC"/>
 </part>
-<part name="X4" library="crystals" library_urn="urn:adsk.eagle:library:20878509" deviceset="TXC-8Y" device="" package3d_urn="urn:adsk.eagle:package:20878596/1"/>
+<part name="X4" library="crystals" library_urn="urn:adsk.eagle:library:20878509" deviceset="TXC-8Y" device="" package3d_urn="urn:adsk.eagle:package:20878596/1">
+<attribute name="FREQ" value="38.4 MHz"/>
+<attribute name="MANUFACTURER" value="TXC"/>
+<attribute name="MPN" value="8Y38472012"/>
+</part>
 <part name="SUPPLY24" library="regulators" deviceset="GND" device=""/>
 <part name="SUPPLY25" library="regulators" deviceset="GND" device=""/>
@@
 </instance>
 <instance part="X4" gate="G$1" x="203.2" y="132.08" smashed="yes" rot="R270">
-<attribute name="NAME" x="208.28" y="134.62" size="1.27" layer="95" rot="R270"/>
+<attribute name="NAME" x="208.28" y="132.08" size="1.27" layer="95"/>
 <attribute name="VALUE" x="208.28" y="134.62" size="1.27" layer="96" rot="R270"/>
+<attribute name="MANUFACTURER" x="203.2" y="132.08" size="1.778" layer="96" rot="R270" display="off"/>
+<attribute name="MPN" x="208.28" y="127.508" size="1.27" layer="96"/>
+<attribute name="FREQ" x="208.28" y="130.048" size="1.27" layer="96"/>
 </instance>
 <instance part="SUPPLY24" gate="G1" x="195.58" y="127" smashed="yes">
