File: hardware/tottag/rev_n/rev_n_v32.sch (EAGLE design)
At the start: 197 parts, among them J1 TC2030-JLINK-NL-2SIDE, J2 TC2030-JLINK-NL-2SIDE, J4 MOLEX-PICO-SPOX-3SIDE, Q1 CSD75207W15, Q2 MOSFET-NCHANNELXFDN-3, U1 APOLLO4_BLUE_PLUS_SOC_KBR, U2 DW3110, U3 BQ24040, U4 BQ51013B, U6 BNO086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

Commit message: rev_n: Updates from DFM review
Parts:
- R13: value 1k -> 2.2k; MPN (none) -> RC0402FR-072K2L; TOL (none) -> 1%
- R15: DIGIKEY RMCF0402JT2K20CT-ND -> (none); MPN RMCF0402JT2K20 -> RC0402FR-072K2L
- RX14: value 1k -> DNP
- renumbered R14 to RX14
Changed lines of the file:
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@@
 <part name="SUPPLY14" library="supply1" library_urn="urn:adsk.eagle:library:371" deviceset="GND" device=""/>
 <part name="R15" library="passives" library_urn="urn:adsk.eagle:library:20904581" deviceset="RESISTOR" device="0402_RES" package3d_urn="urn:adsk.eagle:package:20904668/2" value="2.2k">
-<attribute name="DIGIKEY" value="RMCF0402JT2K20CT-ND"/>
-<attribute name="MPN" value="RMCF0402JT2K20"/>
+<attribute name="MPN" value="RC0402FR-072K2L"/>
 </part>
 <part name="JP2" library="SparkFun-Jumpers" library_urn="urn:adsk.eagle:library:528" deviceset="JUMPER-SMT_3_1-NC_TRACE" device="_SILK" package3d_urn="urn:adsk.eagle:package:39288/1"/>
@@
 </part>
 <part name="SUPPLY39" library="supply1" library_urn="urn:adsk.eagle:library:371" deviceset="GND" device=""/>
-<part name="R13" library="passives" deviceset="RESISTOR" device="0402_RES" value="1k"/>
-<part name="R14" library="passives" deviceset="RESISTOR" device="0402_RES" value="1k"/>
+<part name="R13" library="passives" deviceset="RESISTOR" device="0402_RES" value="2.2k">
+<attribute name="MPN" value="RC0402FR-072K2L"/>
+<attribute name="TOL" value="1%"/>
+</part>
+<part name="RX14" library="passives" deviceset="RESISTOR" device="0402_RES" value="DNP"/>
 <part name="GND6" library="supply1" library_urn="urn:adsk.eagle:library:371" deviceset="GND" device=""/>
 <part name="LS1" library="audio" library_urn="urn:adsk.eagle:library:20947603" deviceset="PUI_SMT-0440-T-2-R" device="" package3d_urn="urn:adsk.eagle:package:21033088/3"/>
@@
 <wire x1="76.2" y1="116.84" x2="137.16" y2="116.84" width="0.127" layer="98" style="shortdash"/>
 <wire x1="76.2" y1="116.84" x2="76.2" y2="149.86" width="0.127" layer="98" style="shortdash"/>
-<text x="77.47" y="148.844" size="0.8128" layer="98" align="top-left">Reference: Datasheet §7.3.13 TS Resistor Network
+<text x="76.962" y="145.288" size="0.6096" layer="98" align="top-left">Reference: Datasheet §7.3.13 TS Resistor Network
 ----
 Properties from the BQ51013B datasheet:
@@
 NTC is 2.97kΩ @ 60ºC
 easy shift is add 2kΩ offset to NTC
-now V_COLD trips when NTC is 26.5kΩ (1.8ºC)</text>
+now V_COLD trips when NTC is 26.5kΩ (1.8ºC)
+----
+Rev N: use 2.2kΩ to reduce BOM count</text>
 <wire x1="76.2" y1="149.86" x2="137.16" y2="149.86" width="0.127" layer="98" style="shortdash"/>
 <wire x1="137.16" y1="116.84" x2="137.16" y2="149.86" width="0.127" layer="98" style="shortdash"/>
@@
 filter</text>
 <text x="110.744" y="128.27" size="0.8128" layer="98" rot="R90" align="top-left">Fig32 NTC</text>
-<text x="87.122" y="122.174" size="0.8128" layer="98" align="top-left">Fig32 R1</text>
-<wire x1="97.79" y1="128.27" x2="82.55" y2="128.27" width="0.127" layer="98" style="shortdash"/>
-<wire x1="82.55" y1="128.27" x2="82.55" y2="120.65" width="0.127" layer="98" style="shortdash"/>
-<wire x1="97.79" y1="128.27" x2="97.79" y2="120.65" width="0.127" layer="98" style="shortdash"/>
-<wire x1="97.79" y1="120.65" x2="82.55" y2="120.65" width="0.127" layer="98" style="shortdash"/>
+<text x="87.884" y="119.634" size="0.8128" layer="98" align="top-left">Fig32 R1</text>
+<wire x1="98.552" y1="128.27" x2="82.042" y2="128.27" width="0.127" layer="98" style="shortdash"/>
+<wire x1="82.042" y1="128.27" x2="82.042" y2="118.364" width="0.127" layer="98" style="shortdash"/>
+<wire x1="98.552" y1="128.27" x2="98.552" y2="118.364" width="0.127" layer="98" style="shortdash"/>
+<wire x1="98.552" y1="118.364" x2="82.042" y2="118.364" width="0.127" layer="98" style="shortdash"/>
 <text x="39.37" y="63.5" size="0.8128" layer="98" align="top-left">ISET controls constant charge current
 Battery wants 0.2C * 1200 mAh = 240 mA
@@
 <attribute name="NAME" x="46.7614" y="85.09" size="1.778" layer="95" rot="R90"/>
 <attribute name="VALUE" x="51.562" y="85.09" size="1.778" layer="96" rot="R90"/>
-<attribute name="DIGIKEY" x="48.26" y="88.9" size="1.27" layer="96" rot="R90" align="top-left" display="off"/>
 <attribute name="MPN" x="48.26" y="88.9" size="1.27" layer="96" rot="R90" align="top-left" display="off"/>
 </instance>
@@
 <attribute name="NAME" x="92.71" y="125.9586" size="1.778" layer="95"/>
 <attribute name="VALUE" x="92.71" y="121.158" size="1.778" layer="96"/>
-</instance>
-<instance part="R14" gate="G$1" x="86.36" y="124.46" smashed="yes">
+<attribute name="MPN" x="96.52" y="124.46" size="1.778" layer="96" display="off"/>
+<attribute name="TOL" x="92.456" y="119.888" size="0.8128" layer="96" display="both"/>
+</instance>
+<instance part="RX14" gate="G$1" x="86.36" y="124.46" smashed="yes">
 <attribute name="NAME" x="82.55" y="125.9586" size="1.778" layer="95"/>
 <attribute name="VALUE" x="82.55" y="121.158" size="1.778" layer="96"/>
@@
 </segment>
 <segment>
-<pinref part="R14" gate="G$1" pin="1"/>
+<pinref part="RX14" gate="G$1" pin="1"/>
 <pinref part="SUPPLY38" gate="1" pin="GND"/>
 <wire x1="81.28" y1="124.46" x2="78.74" y2="124.46" width="0.1524" layer="91"/>
@@
 <segment>
 <pinref part="R13" gate="G$1" pin="1"/>
-<pinref part="R14" gate="G$1" pin="2"/>
+<pinref part="RX14" gate="G$1" pin="2"/>
 <wire x1="91.44" y1="124.46" x2="88.9" y2="124.46" width="0.1524" layer="91"/>
 </segment>
