File: hardware/tottag/rev_n/rev_n v35.sch (EAGLE design)
At the start: 197 parts, among them J1 TC2030-JLINK-NL-2SIDE, J2 TC2030-JLINK-NL-2SIDE, J4 MOLEX-PICO-SPOX-3SIDE, Q1 CSD75207W15, Q2 MOSFET-NCHANNELXFDN-3, U1 APOLLO4_BLUE_PLUS_SOC_KBR, U2 DW3110, U3 BQ24040, U4 BQ51013B, U6 BNO086, U7 QM14068, U8 AS5FXXX04SND, X1 ABM12W, X2 TXC-9HT12, X3 TXC-9HT12

Commit message: rev_n: manufacturing fixes
 - Fix U2 footprint
 - Add tCream for S4
 - Fix AP4/9DOF SPI/I2C mux mismatch with SJ's
    - Removes RX9 and RZ12
 - Rename solder jumpers as SJ#
Parts:
- removed RX9: DNP, passives:RESISTOR0603_RES
- removed RZ12: 0, passives:RESISTOR0402_RES
- added SJ5, SJ6, SJ7: JUMPER-SMT_3_1-NC_TRACE_SILK, SparkFun-Jumpers:JUMPER-SMT_3_1-NC_TRACE_SILK
- renumbered JP1 to SJ1, JP10 to J5, JP11 to J6, JP12 to SJ4, JP2 to SJ2, JP3 to SJ3, JP9 to J3
Connections:
- removed net AP4_GP09/TT_9DOF_H_SDA/H_MISO/TX: RX5.2, U1.GPIO32, U6.H_SDA/H_MISO/TX
- removed net AP4_GP10/TT_9DOF_SA0/H_MOSI: U1.GPIO33, U6.SA0/H_MOSI
- new net 9DOF_H_SDA/H_MISO/TX: RX5.2, SJ5.1, SJ6.2, U6.H_SDA/H_MISO/TX
- new net 9DOF_SA0/H_MOSI: SJ5.2, SJ6.1, U6.SA0/H_MOSI
- new net AP4_GP09/TT_9DOF_H_MOSI: SJ5.3, U1.GPIO32
- new net AP4_GP10/TT_9DOF_H_MISO: SJ6.3, U1.GPIO33
- net +1V8: now also SJ7.3; no longer RZ12.2
- net BNO_PS1: now also SJ7.2; no longer RX9.2, RZ12.1
- net GND: now also SJ7.1; no longer RX9.1
Other:
- note added: "Switch SJ5, SJ6, and SJ7 for I2C"
